File: hardware/conex_focus_flex.brd (EAGLE design)
At the start: 74.9 x 21.8 mm, 0 parts

Commit message: HW: Board cleanup
Routing:
- net GND: track 160.9 -> 160.4 mm
Other:
- board size 74.9 x 21.8 mm -> 74.6 x 21.8 mm
- board text added: "FPC THICKNESS: 0.10mm"
- board text added: "STIFFENER THICKNESS: 0.20MM"
- board text removed: "FPC THICKNESS: 0.15mm"
- board text removed: "STIFFENER THICKNESS: 0.15MM"
