File: hardware/xboxhdmi.brd (EAGLE design)
At the start: 52 x 51 mm, 58 parts, among them J1 5034802000, J2 10029449_HDMI, U1 STM32F070F6P6TR, U2 ADV7511, U3 MIC2091

Commit message: HW: Board cleanup
Parts:
- added 1V8: (no value), my-library:SMD1,27-2,54
- moved CLK 9.41 mm to (35.7, 9.41)
Connections:
- net DVDD: now also 1V8.1
Routing:
- net DVDD: track 56.2 -> 68.9 mm
- net CLK: track 31.1 -> 37.6 mm
- net GND: vias 112 -> 118
Other:
- board text added: "https://github.com/Ryzee119/ XboxHDMI-Ryzee119"
- board text removed: "https://github.com/ Ryzee119/OGXboxHDMI/"
Changed lines of the file:
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@@
 <setting verticaltext="up"/>
 </settings>
-<grid distance="10" unitdist="mil" unit="mil" style="lines" multiple="1" display="yes" altdistance="2.5" altunitdist="mil" altunit="mil"/>
+<grid distance="10" unitdist="mil" unit="mm" style="lines" multiple="1" display="yes" altdistance="2.5" altunitdist="mil" altunit="mm"/>
 <layers>
 <layer number="1" name="Top" color="4" fill="1" visible="yes" active="yes"/>
@@
 <layer number="27" name="tValues" color="7" fill="1" visible="no" active="yes"/>
 <layer number="28" name="bValues" color="7" fill="1" visible="no" active="yes"/>
-<layer number="29" name="tStop" color="7" fill="3" visible="no" active="yes"/>
+<layer number="29" name="tStop" color="7" fill="3" visible="yes" active="yes"/>
 <layer number="30" name="bStop" color="7" fill="6" visible="no" active="yes"/>
 <layer number="31" name="tCream" color="7" fill="4" visible="no" active="yes"/>
@@
 <text x="7.62" y="24.75" size="1.6764" layer="21" rot="R90">Ryzee119
 XboxHDMI</text>
-<text x="29.36875" y="33.9725" size="0.8128" layer="21">https://github.com/
-Ryzee119/OGXboxHDMI/</text>
-<rectangle x1="30.7975" y1="0.15875" x2="32.86125" y2="0.79375" layer="29"/>
+<text x="30.06725" y="34.4805" size="0.6096" layer="21">https://github.com/Ryzee119/
+XboxHDMI-Ryzee119</text>
 <wire x1="0.224" y1="22.7975" x2="0.224" y2="0.47625" width="0.3048" layer="20"/>
 <text x="4.1275" y="-10.4775" size="0.8128" layer="21">DA</text>
@@
 </element>
 <element name="J1" library="my-library" library_urn="urn:adsk.eagle:library:7078210" package="5034802000" package3d_urn="urn:adsk.eagle:package:14718971/2" override_package3d_urn="urn:adsk.eagle:package:12584828/2" override_package_urn="urn:adsk.eagle:footprint:12584829/1" override_locally_modified="yes" value="5034802000" x="3.94775" y="7.775" smashed="yes" rot="R270"/>
-<element name="CLK" library="my-library" library_urn="urn:adsk.eagle:library:7078210" package="SMD1,27-2,54" package3d_urn="urn:adsk.eagle:package:7737318/5" value="" x="36.2" y="0.015" smashed="yes" rot="R90">
-<attribute name="NAME" x="37.2" y="-0.885" size="0.8128" layer="25" rot="R180"/>
-<attribute name="VALUE" x="36.2" y="0.015" size="0.0254" layer="27" rot="R90"/>
+<element name="CLK" library="my-library" library_urn="urn:adsk.eagle:library:7078210" package="SMD1,27-2,54" package3d_urn="urn:adsk.eagle:package:7737318/5" value="" x="35.692" y="9.413" smashed="yes" rot="R90">
+<attribute name="NAME" x="36.692" y="8.513" size="0.8128" layer="25" rot="R180"/>
+<attribute name="VALUE" x="35.692" y="9.413" size="0.0254" layer="27" rot="R90"/>
 </element>
 <element name="LED1" library="led" library_urn="urn:adsk.eagle:library:259" package="CHIP-LED0603" package3d_urn="urn:adsk.eagle:package:15819/3" value="" x="25.0825" y="-11.58875" smashed="yes" rot="R180">
@@
 <attribute name="SPICEPREFIX" value="R" x="8.9535" y="-1.5875" size="1.778" layer="27" rot="R270" display="off"/>
 <attribute name="VALUE" x="7.0485" y="-0.9525" size="1.27" layer="27" rot="R270"/>
+</element>
+<element name="1V8" library="my-library" library_urn="urn:adsk.eagle:library:7078210" package="SMD1,27-2,54" package3d_urn="urn:adsk.eagle:package:7737318/5" value="" x="35.4965" y="-0.254" smashed="yes" rot="R90">
+<attribute name="NAME" x="33.7055" y="0.1525" size="0.8128" layer="25" rot="R180"/>
+<attribute name="VALUE" x="35.4965" y="-0.254" size="0.0254" layer="27" rot="R90"/>
 </element>
 </elements>
@@
 <via x="15.875" y="34.35375" extent="1-16" drill="0.35"/>
 <via x="21.59" y="34.5125" extent="1-16" drill="0.35"/>
-<via x="32.0675" y="34.67125" extent="1-16" drill="0.35"/>
+<via x="30.7975" y="33.90925" extent="1-16" drill="0.35"/>
 <via x="40.9575" y="35.1475" extent="1-16" drill="0.35"/>
 <via x="36.03625" y="32.29" extent="1-16" drill="0.35"/>
@@
 <via x="11.43" y="8.95375" extent="1-16" drill="0.35"/>
 <via x="29.365" y="-0.3175" extent="1-16" drill="0.35"/>
-<via x="31.27375" y="-0.3175" extent="1-16" drill="0.35"/>
-<via x="32.93" y="-0.3175" extent="1-16" drill="0.35"/>
+<via x="30.76575" y="-0.3175" extent="1-16" drill="0.35"/>
 <via x="26.51125" y="-0.635" extent="1-16" drill="0.35"/>
 <via x="24.4475" y="-0.635" extent="1-16" drill="0.35"/>
@@
 <contactref element="J1" pad="P$4"/>
 <contactref element="J1" pad="P$3"/>
-<via x="34.09125" y="6.07125" extent="1-16" drill="0.35"/>
+<via x="34.85325" y="7.34125" extent="1-16" drill="0.35"/>
 <via x="30.91625" y="7.34125" extent="1-16" drill="0.35"/>
 <via x="29.365" y="1.27" extent="1-16" drill="0.35"/>
-<via x="31.27" y="1.27" extent="1-16" drill="0.35"/>
-<via x="32.921" y="1.27" extent="1-16" drill="0.35"/>
+<via x="30.762" y="1.27" extent="1-16" drill="0.35"/>
+<via x="31.905" y="1.27" extent="1-16" drill="0.35"/>
 <contactref element="LED1" pad="C"/>
 <via x="25.55875" y="-13.49375" extent="1-16" drill="0.35"/>
@@
 <via x="1.27" y="2.286" extent="1-16" drill="0.35"/>
 <via x="1.27" y="1.27" extent="1-16" drill="0.35"/>
+<via x="34.85325" y="5.81725" extent="1-16" drill="0.35"/>
+<via x="34.85325" y="4.03925" extent="1-16" drill="0.35"/>
+<via x="33.64675" y="2.64225" extent="1-16" drill="0.35"/>
+<via x="34.85325" y="1.56275" extent="1-16" drill="0.35"/>
+<via x="36.56775" y="4.03925" extent="1-16" drill="0.35"/>
+<via x="36.56775" y="5.81725" extent="1-16" drill="0.35"/>
+<via x="36.56775" y="7.34125" extent="1-16" drill="0.35"/>
 </signal>
 <signal name="PLVDD">
@@
 <wire x1="13.3968" y1="3.4191" x2="14.3165" y2="4.3388" width="0.2" layer="1"/>
 <wire x1="13.3968" y1="2.48348125" x2="13.3968" y2="3.4191" width="0.2" layer="1"/>
+<contactref element="1V8" pad="1"/>
+<wire x1="35.4965" y1="-0.254" x2="33.782" y2="-0.254" width="0.254" layer="1"/>
+<wire x1="33.782" y1="-0.254" x2="33.02" y2="-1.016" width="0.254" layer="1"/>
+<wire x1="33.02" y1="-1.016" x2="28.194" y2="-1.016" width="0.254" layer="1"/>
+<wire x1="28.194" y1="-1.016" x2="26.924" y2="0.254" width="0.254" layer="1"/>
+<wire x1="26.924" y1="0.254" x2="26.924" y2="0.762" width="0.254" layer="1"/>
+<wire x1="27.686" y1="1.524" x2="27.94" y2="1.524" width="0.254" layer="1"/>
+<wire x1="27.94" y1="1.524" x2="28.2575" y2="1.8415" width="0.254" layer="1"/>
+<wire x1="28.2575" y1="1.8415" x2="28.2575" y2="2.80125" width="0.254" layer="1"/>
+<wire x1="26.924" y1="0.762" x2="27.686" y2="1.524" width="0.254" layer="1"/>
 </signal>
 <signal name="AVDD">
@@
 <contactref element="CLK" pad="1"/>
 <contactref element="R17" pad="2"/>
-<wire x1="36.2" y1="0.015" x2="34.46909375" y2="0.015" width="0.6096" layer="1"/>
-<wire x1="34.46909375" y1="0.015" x2="34.00784375" y2="0.47625" width="0.6096" layer="1"/>
-<wire x1="34.00784375" y1="0.47625" x2="28.2575" y2="0.47625" width="0.6096" layer="1"/>
+<wire x1="35.692" y1="9.413" x2="35.692" y2="3.571" width="0.6096" layer="1"/>
+<wire x1="35.692" y1="3.571" x2="32.59725" y2="0.47625" width="0.6096" layer="1"/>
+<wire x1="28.2575" y1="0.47625" x2="32.59725" y2="0.47625" width="0.6096" layer="1"/>
 <wire x1="8.9535" y1="-2.4375" x2="11.1125" y2="-2.4375" width="0.6096" layer="1"/>
 <wire x1="11.1125" y1="-2.4375" x2="11.215" y2="-2.54" width="0.6096" layer="1"/>
