File: hardware/xboxhdmi.sch (EAGLE design)
At the start: 58 parts, among them J1 5034802000, J2 10029449_HDMI, U1 STM32F070F6P6TR, U2 ADV7511, U3 MIC2091

Commit message: HW: Remove old notes
Other:
- note added: "VCC=1V8"
- note removed: "100uF capacitor 493-14561-6-ND"
- note removed: "10uf capacitor C3216X5R1C106M"
- note removed: "1V8"
- note removed: "Inductor: TDK MPZ1608S221A"
- note removed: "Temp Notes:"
Changed lines of the file:
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@@
 <sheet>
 <plain>
-<text x="276.86" y="195.58" size="1.778" layer="91">Inductor:
-TDK MPZ1608S221A</text>
-<text x="276.86" y="187.96" size="1.778" layer="91">10uf capacitor
-C3216X5R1C106M</text>
-<text x="205.74" y="147.32" size="1.778" layer="91">1V8</text>
-<text x="276.86" y="180.34" size="1.778" layer="91">100uF capacitor
-493-14561-6-ND</text>
+<text x="198.12" y="149.86" size="1.778" layer="97">VCC=1V8</text>
 <text x="146.05" y="1.27" size="1.778" layer="97">5V supply to HDMI Connector
 Current limited to 100mA with MIC2091
@@
 <text x="69.85" y="208.28" size="2.54" layer="97">HDMI CONTROLLER</text>
 <text x="68.58" y="147.32" size="2.54" layer="97">HDMI BRIDGE</text>
-<text x="276.86" y="203.2" size="1.778" layer="91">Temp Notes:</text>
 <text x="-49.53" y="111.76" size="2.54" layer="97" rot="R90" align="bottom-right">Molex
 0151660207

Commit message: HW: Board cleanup
Parts:
- added 1V8: (no value), my-library:SMD2
Connections:
- net DVDD: now also 1V8.P
Other:
- note added: "XboxHDMI-Ryzee119"
- note added: "https://github.com/Ryzee119/XboxHDMI-Ryzee119"
- note removed: "VCC=1.8V"
- note removed: "https://github.com/Ryzee119/OGXboxHDMI"
- note removed: "ogXboxHDMI"
Changed lines of the file:
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@@
 <part name="GND18" library="supply1" library_urn="urn:adsk.eagle:library:371" deviceset="GND" device=""/>
 <part name="GND20" library="supply1" library_urn="urn:adsk.eagle:library:371" deviceset="GND" device=""/>
+<part name="1V8" library="my-library" library_urn="urn:adsk.eagle:library:7078210" deviceset="SMD2" device="" package3d_urn="urn:adsk.eagle:package:7737318/5"/>
 </parts>
 <sheets>
@@
 Provides reverse current protection
 Meets HDMI 5V Source Requirement</text>
-<text x="260.35" y="-25.4" size="2.54" layer="94">ogXboxHDMI</text>
+<text x="260.35" y="-25.4" size="2.54" layer="94">XboxHDMI-Ryzee119</text>
 <text x="260.35" y="-30.48" size="2.54" layer="94">August 2019</text>
 <text x="260.35" y="-20.32" size="2.54" layer="94">BY RYZEE119</text>
@@
 <rectangle x1="222.1484" y1="-20.1168" x2="223.774" y2="-20.0152" layer="94"/>
 <text x="297.18" y="-13.97" size="1.9304" layer="94" align="center-right">Original Xbox 100% Digital HDMI</text>
-<text x="297.18" y="-10.16" size="1.9304" layer="94" align="center-right">https://github.com/Ryzee119/OGXboxHDMI</text>
+<text x="297.18" y="-10.16" size="1.9304" layer="94" align="center-right">https://github.com/Ryzee119/XboxHDMI-Ryzee119</text>
 <text x="123.19" y="170.18" size="1.778" layer="97">SWD Programming
 Header</text>
 <text x="217.17" y="171.45" size="1.778" layer="97">5V to 3.3V@150mA
 5V to 1.8V@150mA</text>
-<text x="279.4" y="210.82" size="1.778" layer="97">VCC=1.8V</text>
 <text x="213.36" y="208.28" size="2.54" layer="97">POWER SUPPLIES</text>
 <text x="69.85" y="208.28" size="2.54" layer="97">HDMI CONTROLLER</text>
@@
 <instance part="GND20" gate="1" x="-7.62" y="-15.24" smashed="yes">
 <attribute name="VALUE" x="-10.16" y="-17.78" size="1.778" layer="96"/>
+</instance>
+<instance part="1V8" gate="1" x="139.7" y="128.27" smashed="yes" rot="R270">
+<attribute name="VALUE" x="136.398" y="129.413" size="1.778" layer="96" rot="R270"/>
 </instance>
 </instances>
@@
 <junction x="124.46" y="116.84"/>
 <pinref part="C15" gate="G$1" pin="1"/>
-<wire x1="129.54" y1="124.46" x2="132.08" y2="124.46" width="0.1524" layer="91"/>
 <wire x1="132.08" y1="124.46" x2="139.7" y2="124.46" width="0.1524" layer="91"/>
-<wire x1="139.7" y1="124.46" x2="147.32" y2="124.46" width="0.1524" layer="91"/>
-<wire x1="147.32" y1="124.46" x2="154.94" y2="124.46" width="0.1524" layer="91"/>
-<wire x1="154.94" y1="124.46" x2="162.56" y2="124.46" width="0.1524" layer="91"/>
+<wire x1="139.7" y1="124.46" x2="162.56" y2="124.46" width="0.1524" layer="91"/>
 <wire x1="162.56" y1="124.46" x2="177.8" y2="124.46" width="0.1524" layer="91"/>
 <wire x1="177.8" y1="124.46" x2="180.34" y2="124.46" width="0.1524" layer="91"/>
@@
 <label x="129.54" y="124.46" size="1.778" layer="95"/>
 <wire x1="124.46" y1="121.92" x2="127" y2="124.46" width="0.1524" layer="91"/>
-<wire x1="127" y1="124.46" x2="129.54" y2="124.46" width="0.1524" layer="91"/>
+<wire x1="127" y1="124.46" x2="132.08" y2="124.46" width="0.1524" layer="91"/>
+<pinref part="1V8" gate="1" pin="P"/>
+<wire x1="139.7" y1="125.73" x2="139.7" y2="124.46" width="0.1524" layer="91"/>
 </segment>
 </net>
@@
 <pinref part="U2" gate="G$1" pin="AVDD@1"/>
 <pinref part="C14" gate="G$1" pin="1"/>
-<wire x1="129.54" y1="139.7" x2="132.08" y2="139.7" width="0.1524" layer="91"/>
 <wire x1="132.08" y1="139.7" x2="139.7" y2="139.7" width="0.1524" layer="91"/>
 <wire x1="139.7" y1="139.7" x2="147.32" y2="139.7" width="0.1524" layer="91"/>
@@
 <label x="129.54" y="139.7" size="1.778" layer="95"/>
 <wire x1="124.46" y1="137.16" x2="127" y2="139.7" width="0.1524" layer="91"/>
-<wire x1="127" y1="139.7" x2="129.54" y2="139.7" width="0.1524" layer="91"/>
+<wire x1="127" y1="139.7" x2="132.08" y2="139.7" width="0.1524" layer="91"/>
 </segment>
 </net>
